Commit message: Add prismatic joint

File: urdf/ur_macro.xacro (robot description, xacro)
@@ -132,5 +132,18 @@
     <!-- Placeholder for ros2_control transmission which don't yet exist -->
     <!-- links -  main serial chain -->
-    <link name="${tf_prefix}base_link"/>
+    <link name="${tf_prefix}base_link">
+          <inertial>
+        <mass value="${shoulder_mass}"/>
+        <origin rpy="${shoulder_inertia_rotation}" xyz="${shoulder_cog}"/>
+        <inertia
+            ixx="${shoulder_inertia_ixx}"
+            ixy="${shoulder_inertia_ixy}"
+            ixz="${shoulder_inertia_ixz}"
+            iyy="${shoulder_inertia_iyy}"
+            iyz="${shoulder_inertia_iyz}"
+            izz="${shoulder_inertia_izz}"
+        />
+      </inertial>
+    </link>
     <link name="${tf_prefix}base_link_inertia">
       <visual>
@@ -321,5 +334,5 @@
     </joint>
     <!-- joints - main serial chain -->
-    <joint name="${tf_prefix}base_link-base_link_inertia" type="fixed">
+    <joint name="${tf_prefix}prismatic_joint" type="prismatic">
       <parent link="${tf_prefix}base_link" />
       <child link="${tf_prefix}base_link_inertia" />
@@ -329,4 +342,7 @@
            link/frame) to introduce the necessary rotation over Z (of pi rad).
       -->
+       <limit lower="0.0" upper="1.0" effort="10" velocity="10"/>
+      <dynamics damping="0" friction="0"/>
+      <axis xyz="0 0 1" />
       <origin xyz="0 0 0" rpy="0 0 ${pi}" />
     </joint>
