Commit message: Cleanup

File: urdf/ur.ros2_control.xacro (robot description, xacro)
@@ -65,4 +65,14 @@
         </xacro:unless>
       </hardware>
+      <joint name="${tf_prefix}prismatic_joint">
+        <command_interface name="position"/>
+        <command_interface name="velocity"/>
+        <state_interface name="position">
+          <!-- initial position for the FakeSystem and simulation -->
+          <param name="initial_value">${initial_positions['prismatic_joint']}</param>
+        </state_interface>
+        <state_interface name="velocity"/>
+        <state_interface name="effort"/>
+      </joint>
       <joint name="${tf_prefix}shoulder_pan_joint">
         <command_interface name="position"/>
